File: Kicad/DOTApad.kicad_sch (KiCad schematic)
At the start: 0 parts

Commit message: made schematic
Parts:
- added D1, D10, D11, D12, D2, D3, D4, D5, D6, D7, D8, D9: D, Diode_THT:D_DO-35_SOD27_P7.62mm_Horizontal, symbol Device:D
- added SW1, SW10, SW11, SW12, SW2, SW3, SW4, SW5, SW6, SW7, SW8, SW9: SW_Push, Button_Switch_Keyboard:SW_Cherry_MX_1.00u_PCB, symbol Switch:SW_Push
- added U1: MOUDLE-SEEEDUINO-XIAO, RF_Module:MCU_Seeed_ESP32C3, symbol XIAO_RP2040:MOUDLE-SEEEDUINO-XIAO
- added U3: ER_OLEDM0.91_1x-I2C, Display:ER_OLEDM0.91_1x-I2C, symbol Display_Graphic:ER_OLEDM0.91_1x-I2C
Connections:
- new net: D8.2 (A), SW8.2
- new net: D6.2 (A), SW6.2
- new net: D9.2 (A), SW9.2
- new net: D10.2 (A), SW10.2
- new net: D5.2 (A), SW5.2
- new net: D1.2 (A), SW1.2
- new net: D12.2 (A), SW12.2
- new net: D3.2 (A), SW3.2
- new net: D11.2 (A), SW11.2
- new net: D7.2 (A), SW7.2
- new net: D4.2 (A), SW4.2
- new net: D2.2 (A), SW2.2
- new net GND: U1.13 (GND), U3.1 (GND)
- new net GP1: D1.1 (K), D2.1 (K), D3.1 (K), D4.1 (K), D5.1 (K), D6.1 (K), D7.1 (K), D8.1 (K), SW1.1, SW5.1, SW9.1, U1.1 (PA02_A0_D0), U1.8 (PB09_A7_D7_RX), U1.9 (PA7_A8_D8_SCK)
- new net GP10: D10.1 (K), D11.1 (K), D12.1 (K), D9.1 (K), SW10.1, SW11.1, SW12.1, SW2.1, SW3.1, SW4.1, SW6.1, SW7.1, SW8.1, U1.10 (PA5_A9_D9_MISO), U1.2 (PA4_A1_D1), U1.3 (PA10_A2_D2), U1.4 (PA11_A3_D3)
- new net SCL: U1.6 (PA9_A5_D5_SCL), U3.3 (SCL)
- new net SDA: U1.5 (PA8_A4_D4_SDA), U3.4 (SDA)
- new net VCC: U1.14 (5V), U3.2 (VCC)
Other:
- note added: "OLED Display Pins"
- note added: "Swiches"
